File: hardware/eagle_project/SolarPowerBoard/SolarPowerBoard.brd (EAGLE design)
At the start: 160 x 100 mm, 74 parts, among them IC1 BQ29700DSET, IC3 TPS63031DSKT, J2 105017-0001, Q3 FDN302P, U4 MCP73831T-2ACI/OT

Commit message: First version new PCB added
Parts:
- removed JP2: JUMPER-SMT_3_1-NC_TRACE_NO-SILK, SparkFun-Jumpers:SMT-JUMPER_3_1-NC_TRACE_NO-SILK
- removed R19, R20: 0.3, SparkFun-Resistors:0805
- added J5: XG8S-0331, XG8S-0331:HDRV3W70P0X254_1X3_760X280X680
- added K1: G6E-134P-US_DC5, G6E-134P-US_DC5:DIP762W60P254L1595H800Q12N
- added RGPIO1, RGPIO2, RGPIO3, RGPIO4: (no value), SparkFun-Resistors:0603
- C3: value 10uF -> 10UF
- L1: value 27µH/±20%/3.3A -> SRR1280-270M; device SparkFun-Coils:INDUCTOR_SDR1307 -> SolarPowerBoard:IND_BOURNS_SRR1280
- moved SCL_SDA 157.1 mm to (64.8, 18.6), turned to 90 degrees
- moved D5 149.6 mm to (37.7, 41.0), turned to 180 degrees
- moved RLED1 149.4 mm to (37.0, 38.9), turned to 90 degrees
- moved RX_TX 149.1 mm to (64.8, 24.3), flipped to the bottom, turned to 90 degrees
- moved R23 145.2 mm to (53.6, 40.8), turned to 90 degrees
- moved SDA 144.6 mm to (56.8, 19.4), turned to 180 degrees
- moved R25 143.2 mm to (44.7, 43.3), turned to 90 degrees
- moved J2 139.9 mm to (66.6, 39.0), turned to 90 degrees
- moved SCL 138.4 mm to (56.8, 23.3)
- moved R14 137.8 mm to (63.1, 46.9)
- moved R24 137.7 mm to (41.3, 39.4), turned to 90 degrees
- moved L3 132.8 mm to (56.1, 33.7), turned to 180 degrees
- moved C11 126.9 mm to (41.9, 33.8), turned to 270 degrees
- moved C12 124.3 mm to (35.4, 34.2), turned to 180 degrees
- moved RCG3 122.6 mm to (23.0, 32.4), turned to 180 degrees
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Connections:
- removed net ALM_FG: R19.1, RB2.DIO22
- removed net RSTIO_FG: R20.2, RB2.RESET
- removed net SOURCE_OUTPUT: C12.1, C2.1, COUT2.2, IC3.5, JP2.1, R1.1, RCG3.1, RF2.2, RS1.2, U$3.10, U4.3
- new net N$18: L1.1, U$1.3
- new net N$20: C12.1, K1.12, U4.3
- new net N$28: RB2.MOSI, RGPIO1.1
- new net N$30: RB2.MISO, RGPIO2.1
- new net N$33: RB2.BTN1, RGPIO3.1
- new net N$41: RB2.BTN2, RGPIO4.1
- new net POWER_INPUT: C2.1, IC3.5, K1.7, RCG3.1, U$3.10
- new net SOLAR_OUTPUT: COUT2.2, J5.1, K1.10, R1.1, RF2.2, RS1.2
- net GPIO1: now also RGPIO1.2; no longer RB2.NC@3
- net GPIO2: now also RGPIO2.2; no longer RB2.NC@2
- net GPIO3: now also RGPIO3.2; no longer RB2.NC@1
- net GPIO4: now also RGPIO4.2; no longer RB2.NC
- net N$1: now also J5.3, L1.2; no longer JP2.3, L1.P$1
- net N$16: now also J5.2; no longer JP2.2
- net N$23: now also K1.6; no longer L1.P$2, U$1.3
- net VDD: no longer R19.2, R20.1
- net VDD_CHARGER: now also K1.1
Routing:
- net GND: track 0.00 -> 110.0 mm, vias 0 -> 44
- net PO.22(CTS)-DIO18(RTS): track 0.00 -> 99.2 mm, vias 0 -> 1
- net PO.23(RTS)-DIO19(CTS): track 0.00 -> 78.4 mm, vias 0 -> 3
- net N$36: track 0.00 -> 76.3 mm, vias 0 -> 1
- net VDD: track 0.00 -> 70.8 mm, vias 0 -> 2
- net N$37: track 0.00 -> 68.4 mm, vias 0 -> 1
- net SDA_FG: track 0.00 -> 65.2 mm
- net SCL_FG: track 0.00 -> 63.8 mm, vias 0 -> 4
- net PO.24(TX)-DIO2(RX): track 0.00 -> 63.8 mm, vias 0 -> 2
- net N$40: track 0.00 -> 63.4 mm, vias 0 -> 1
- net N$38: track 0.00 -> 56.1 mm, vias 0 -> 1
- net SOLAR_OUTPUT: track 0.00 -> 55.7 mm, vias 0 -> 2
- net N$41: track 0.00 -> 54.5 mm
- net N$39: track 0.00 -> 53.1 mm, vias 0 -> 1
- net PO.25(RX)-DIO3(TX): track 0.00 -> 52.4 mm, vias 0 -> 2
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- added copper zone on layer 16, net AAAA
- added copper zone on layer 1, net AFDV
- added copper zone on layer 1, net BAAB
- added copper zone on layer 1, net BOH
- added copper zone on layer 1, net GND
- added copper zone on layer 16, net GND
Other:
- board size 160 x 100 mm -> 68.8 x 53.6 mm
- board text added: "DIRECT"
- board text added: "Harvester"
- board text added: "IN"
- board text added: "RX"
- board text added: "SCL"
- board text added: "SDA"
- board text added: "TX"
- board text added: "USB-CHARGING"
