File: hardware/eagle_project/SolarPowerBoard/SolarPowerBoard.sch (EAGLE design)
At the start: 74 parts, among them IC1 BQ29700DSET, IC3 TPS63031DSKT, J2 105017-0001, Q3 FDN302P, U4 MCP73831T-2ACI/OT

Commit message: First version new PCB added
Parts:
- removed JP2: JUMPER-SMT_3_1-NC_TRACE_NO-SILK, SparkFun-Jumpers:JUMPER-SMT_3_1-NC_TRACE_NO-SILK
- removed R19, R20: 0.3, SparkFun-Resistors:0.3OHM-0805-1/8W-1%
- added J5: XG8S-0331, XG8S-0331:XG8S-0331
- added K1: G6E-134P-US_DC5, G6E-134P-US_DC5:G6E-134P-US_DC5
- added RGPIO1, RGPIO2, RGPIO3, RGPIO4: (no value), SparkFun-Resistors:RESISTOR0603
- C3: value 10uF -> 10UF
- L1: value 27µH/±20%/3.3A -> SRR1280-270M; device SparkFun-Coils:INDUCTOR-SDR13-27UH -> SolarPowerBoard:SRR1280-270M; OC_NEWARK unknown -> (none)
Connections:
- removed net ALM_FG: R19.1, RB2.DIO22
- removed net RSTIO_FG: R20.2, RB2.RESET
- removed net SOURCE_OUTPUT: C12.1, C2.1, COUT2.2, IC3.VIN, JP2.1, R1.1, RCG3.1, RF2.2, RS1.22, U$3.CSPH, U4.VBAT
- new net N$18: L1.1, U$1.LX
- new net N$20: C12.1, K1.NO, U4.VBAT
- new net N$28: RB2.MOSI, RGPIO1.1
- new net N$30: RB2.MISO, RGPIO2.1
- new net N$33: RB2.BTN1, RGPIO3.1
- new net N$41: RB2.BTN2, RGPIO4.1
- new net POWER_INPUT: C2.1, IC3.VIN, K1.COM, RCG3.1, U$3.CSPH
- new net SOLAR_OUTPUT: COUT2.2, J5.1, K1.NC, R1.1, RF2.2, RS1.22
- net GPIO1: now also RGPIO1.2; no longer RB2.NC@3
- net GPIO2: now also RGPIO2.2; no longer RB2.NC@2
- net GPIO3: now also RGPIO3.2; no longer RB2.NC@1
- net GPIO4: now also RGPIO4.2; no longer RB2.NC
- net N$1: now also J5.3, L1.2; no longer JP2.3, L1.1
- net N$16: now also J5.2; no longer JP2.2
- net N$23: now also K1.GND; no longer L1.2, U$1.LX
- net VDD: no longer R19.2, R20.1
- net VDD_CHARGER: now also K1.5V
Other:
- moved on the sheet: C1-1, C1-2, C10, C7, J1, JP1, RCG3, RTEMP, U$3
