File: hardware/eagle_project/SolarPowerBoard/SolarPowerBoard.sch (EAGLE design)
At the start: 83 parts, among them J2 105017-0001_105017-0001, J3 BAT_ID, J5 XG8S-0331_XG8S-0331, K1 G6E-134P-US_DC5_G6E-134P-US_D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, Q1 SOLARCOMPONENTS_CSD16406Q3, Q2 SOLARCOMPONENTS_CSD16406Q3, Q3 DAVIDE_FDN302P, U1 SOLARCOMPONENTS_SVP1040, U2 SOLARCOMPONENTS_MAX17260, U3 FT230XQ_FT230XQ_2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

Commit message: Hardware: reset out pin now can be routed to DIO22 instead of DIO1 which is reserved for the rf switch on cc1350 launchpads
Parts:
- removed R15: 0, SolarPowerBoard:SPARKFUN-RESISTORS_0.3OHM
- added RES_SEL: POWERSOL_JUMPER-SMT_3_0_SILK, SolarPowerBoard:POWERSOL_JUMPER-SMT_3_0_SILK
- RGPIO1, RGPIO2, RGPIO3, RGPIO4: value 1k -> DNM
Connections:
- removed net DIO1-RESET: B1.DIO1-RESET, R15.2
- removed net N$40: B2.DIO1-RESET, R15.1
- new net DIO1_RESERVED: B1.DIO1-RESET, RES_SEL.3
- new net DIO22: B1.DIO22, RES_SEL.1
- new net NRF_RESET: B2.DIO1-RESET, RES_SEL.2
- net VDD: now also B2.VDD@2; no longer B2.VDD
Other:
- moved on the sheet: RGPIO1, RGPIO2, RGPIO3
